File: hw/sch_pcb/SPACEDOS01A_PCB01A.kicad_pcb (KiCad board)
At the start: 2 copper layers, 90.9 x 50.3 mm, 111 parts, among them J1 HEADER_2x01_PARALLEL, J19 HEADER_2x01_PARALLEL, J2 HEADER_2x01_PARALLEL, J22 HEADER_2x03, J3 HEADER_2x01_PARALLEL, J4 HEADER_1x01, J5 HEADER_1x01, J6 HEADER_1x01, J7 HEADER_1x01, M1 HOLE, M2 HOLE, M3 HOLE, M4 HOLE, M6 BMI-S-210-F, M7 BMI-S-210-F, U1 OPA2314, U10 ATMEGA1284P-AU, U11 PCF85263A, U2 OPA2314, U3 ISL21080DIH312Z-TK 1V25, U4 TS7211, U5 TS5A4594, U6 TPS613221ADBV, U8 TPS613222ADBV, Y1 16MHz, Y2 ABS07-120-32.768KHZ-T

Commit message: edit
Parts:
- removed D4: HLMP-K150+FIX-LED-313, Mlab_D:LED_1206
- removed R26: 2k2, Mlab_R:SMD-0805
- J22: footprint Mlab_Pin_Headers:Straight_2x03 -> Mlab_Pin_Headers:SMD_2x03; moved to B.Cu
- moved J4 3.59 mm to (85.0, -36.1)
- moved J7 3.59 mm to (87.5, -33.5)
- moved R23 2.04 mm to (50.6, -31.0), turned to 0 degrees
- moved J22 1.53 mm to (51.4, -26.2), turned to 0 degrees
- moved C34 0.95 mm to (53.2, -31.8)
Connections:
- U10 pad 21: /cpu/LED -> (no net)
Routing:
- net GND: track 102.3 -> 132.3 mm, vias 172 -> 195
- net PA1: track 94.9 -> 104.0 mm, vias 4 -> 2
- net /cpu/LED: track 7.59 -> 0.00 mm
- net /cpu/PB6: track 3.52 -> 8.97 mm, vias 0 -> 2
- net /cpu/TX0: track 28.3 -> 32.0 mm, vias 1 -> 2
- net /cpu/PB5: track 7.18 -> 5.04 mm
- net Net-(D4-Pad2): track 1.87 -> 0.00 mm
- net /cpu/PB7: track 6.39 -> 8.25 mm
- net /cpu/PC7: track 21.1 -> 20.3 mm
- net /cpu/RX0: track 28.3 -> 29.1 mm, vias 1 -> 2
- net /cpu/PC3: track 22.0 -> 21.4 mm
