File: hw/sch_pcb/cpu.sch (KiCad schematic (older format))
At the start: 29 parts, among them J19 HEADER_2x01_PARALLEL, J22 HEADER_2x03, J4 HEADER_1x01, J5 HEADER_1x01, J6 HEADER_1x01, J7 HEADER_1x01, U10 ATMEGA1284P-AU, U11 PCF85263A, Y1 16MHz, Y2 ABS07-120-32.768KHZ-T

Commit message: edit
Parts:
- removed D4: HLMP-K150+FIX-LED-313, Mlab_D:LED_1206, symbol SPACEDOS01A_PCB01A-rescue:LED-device-DATALOGGER01A-rescue-CCP2019V01A-rescue
- removed R26: 2k2, Mlab_R:SMD-0805, symbol SPACEDOS01A_PCB01A-rescue:R-device-DATALOGGER01A-rescue-CCP2019V01A-rescue
- J22: footprint Mlab_Pin_Headers:Straight_2x03 -> Mlab_Pin_Headers:SMD_2x03
Connections:
- net LED: no longer names the net of U10.21 ((PCINT18/TCK)PC2)
- no-connect marks 23 -> 24
Changed lines of the file:
@@
 EESchema Schematic File Version 4
 LIBS:SPACEDOS01A_PCB01A-cache
-EELAYER 26 0
+EELAYER 29 0
 EELAYER END
 $Descr A4 11693 8268
@@
 	2400 1900 2400 2300
 $Comp
-L SPACEDOS01A_PCB01A-rescue:LED-device-DATALOGGER01A-rescue-CCP2019V01A-rescue D4
-U 1 1 5B2AFFF7
-P 9650 1300
-F 0 "D4" H 9600 1550 50  0000 R CNN
-F 1 "HLMP-K150+FIX-LED-313" H 9800 1450 50  0000 R CNN
-F 2 "Mlab_D:LED_1206" H 9650 1300 50  0001 C CNN
-F 3 "~" H 9650 1300 50  0001 C CNN
-	1    9650 1300
-	0    -1   -1   0
-$EndComp
-$Comp
-L power:GND #PWR0128
-U 1 1 5B2B6028
-P 9650 1550
-F 0 "#PWR0128" H 9650 1300 50  0001 C CNN
-F 1 "GND" H 9655 1377 50  0000 C CNN
-F 2 "" H 9650 1550 50  0001 C CNN
-F 3 "" H 9650 1550 50  0001 C CNN
-	1    9650 1550
-	1    0    0    -1
-$EndComp
-$Comp
 L power:GND #PWR0129
 U 1 1 5B2B60EB
@@
 Wire Wire Line
 	5750 5250 5850 5250
-$Comp
-L SPACEDOS01A_PCB01A-rescue:R-device-DATALOGGER01A-rescue-CCP2019V01A-rescue R26
-U 1 1 5B2CE6CA
-P 9650 950
-F 0 "R26" V 9550 850 50  0000 C CNN
-F 1 "2k2" V 9650 950 50  0000 C CNN
-F 2 "Mlab_R:SMD-0805" V 9580 950 50  0001 C CNN
-F 3 "" H 9650 950 50  0001 C CNN
-	1    9650 950
-	-1   0    0    1
-$EndComp
-Wire Wire Line
-	9650 800  9650 700
-Text Label 6950 3500 0    60   ~ 0
-LED
-Text Label 9650 700  0    60   ~ 0
-LED
-Wire Wire Line
-	9650 1550 9650 1450
-Wire Wire Line
-	9650 1150 9650 1100
 Text Label 6950 3000 0    60   ~ 0
 PB6
@@
 F 0 "J22" H 5900 6441 60  0000 C CNN
 F 1 "HEADER_2x03" H 5900 6441 60  0001 C CNN
-F 2 "Mlab_Pin_Headers:Straight_2x03" H 5900 6300 60  0001 C CNN
+F 2 "Mlab_Pin_Headers:SMD_2x03" H 5900 6300 60  0001 C CNN
 F 3 "" H 5900 6300 60  0000 C CNN
 	1    5900 6200
@@
 Wire Wire Line
 	6850 4000 7200 4000
-Wire Wire Line
-	6850 3500 6950 3500
 NoConn ~ 6850 2800
+NoConn ~ 6850 3500
 $EndSCHEMATC
