File: hw/sch_pcb/SPACEDOS01A_PCB01A/SPACEDOS01A_PCB01A.kicad_pcb (KiCad board)
At the start: 2 copper layers, 90.9 x 50.3 mm, 109 parts, among them J1 HEADER_2x01_PARALLEL, J19 HEADER_2x01_PARALLEL, J2 HEADER_2x01_PARALLEL, J22 HEADER_2x03, J3 HEADER_2x01_PARALLEL, J4 HEADER_1x01, J5 HEADER_1x01, J6 HEADER_1x01, J7 HEADER_1x01, M1 HOLE, M2 HOLE, M3 HOLE, M4 HOLE, M6 BMI-S-210-F, M7 BMI-S-210-F, U1 OPA2314, U10 ATMEGA1284P-AU, U11 PCF85263A, U2 OPA2314, U3 ISL21080DIH312Z-TK 1V25, U4 TS7211, U5 TS5A4594, U6 TPS613221ADBV, U8 TPS613222ADBV, Y1 16MHz, Y2 ABS07-120-32.768KHZ-T

Commit message: edit
Parts:
- added M5: BMI-S-210-F, Mlab_Mechanical:BMI-S-210-F, F.Cu at (36.6, -41.1)
- added M8: BMI-S-204-F, RF_Shielding:Laird_Technologies_BMI-S-204-F_32.00x32.00mm, F.Cu at (17.3, -25.4)
- Y1: footprint Mlab_XTAL:Crystal_HC49-U_Vertical -> Mlab_XTAL:Crystal_HC49-4H_Vertical
- moved Y1 2.54 mm to (50.3, -34.5)
Connections:
- U10 pad 11: Net-(U10-Pad11) -> (no net)
- U10 pad 12: Net-(U10-Pad12) -> (no net)
- U10 pad 13: Net-(U10-Pad13) -> (no net)
- U10 pad 14: Net-(U10-Pad14) -> (no net)
- U10 pad 15: Net-(U10-Pad15) -> (no net)
- U10 pad 16: Net-(U10-Pad16) -> (no net)
- U10 pad 21: Net-(U10-Pad21) -> (no net)
- U10 pad 23: Net-(U10-Pad23) -> (no net)
- U10 pad 24: Net-(U10-Pad24) -> (no net)
- U10 pad 25: Net-(U10-Pad25) -> (no net)
- U10 pad 30: Net-(U10-Pad30) -> (no net)
- U10 pad 31: Net-(U10-Pad31) -> (no net)
- U10 pad 32: Net-(U10-Pad32) -> (no net)
- U10 pad 33: Net-(U10-Pad33) -> (no net)
- U10 pad 34: Net-(U10-Pad34) -> (no net)
- U10 pad 35: Net-(U10-Pad35) -> (no net)
- U10 pad 41: Net-(U10-Pad41) -> (no net)
- U10 pad 42: Net-(U10-Pad42) -> (no net)
- U10 pad 43: Net-(U10-Pad43) -> (no net)
- U10 pad 44: Net-(U10-Pad44) -> (no net)
- U11 pad 4: Net-(U11-Pad4) -> (no net)
- U11 pad 8: Net-(U11-Pad8) -> (no net)
- U11 pad 9: Net-(U11-Pad9) -> (no net)
Routing:
- net PB0: track 1.94 -> 25.1 mm, vias 0 -> 2
- net GND: track 132.3 -> 133.6 mm, vias 195 -> 193
