File: hw/sch_pcb/SPACEDOS01A_PCB01A/SPACEDOS01A_PCB01A.sch (KiCad schematic (older format))
At the start: 51 parts, among them M1 HOLE, M2 HOLE, M3 HOLE, M4 HOLE, M6 BMI-S-210-F, M7 BMI-S-210-F, U1 OPA2314, U2 OPA2314, U3 ISL21080DIH312Z-TK 1V25, U4 TS7211, U5 TS5A4594

Commit message: Edit
Connections:
- net PB0: now reaches R12.1, U5.4 (IN)
Changed lines of the file:
@@
 EESchema Schematic File Version 4
 LIBS:SPACEDOS01A_PCB01A-cache
-EELAYER 29 0
+EELAYER 26 0
 EELAYER END
 $Descr A4 11693 8268
@@
 Wire Wire Line
 	9600 650  10000 650
+Wire Wire Line
+	8350 5150 10550 5150
+Connection ~ 8350 5150
+Text Label 10000 5150 0    60   ~ 0
+Trace
+Text GLabel 10550 5150 2    60   Input ~ 0
+PB0
 $EndSCHEMATC

Commit message: edit
Parts:
- added M5: BMI-S-210-F, Mlab_Mechanical:BMI-S-210-F, symbol MLAB_MECHANICAL:HOLE
- added M8: BMI-S-204-F, RF_Shielding:Laird_Technologies_BMI-S-204-F_32.00x32.00mm, symbol MLAB_MECHANICAL:HOLE
Connections:
- net GND: now also M5.1, M8.1
Changed lines of the file:
@@
 Text GLabel 10550 5150 2    60   Input ~ 0
 PB0
+$Comp
+L MLAB_MECHANICAL:HOLE M5
+U 1 1 5C7015D6
+P 9400 750
+F 0 "M5" V 9300 750 60  0000 C CNN
+F 1 "BMI-S-210-F" H 9400 650 60  0001 C CNN
+F 2 "Mlab_Mechanical:BMI-S-210-F" H 9400 750 60  0001 C CNN
+F 3 "" H 9400 750 60  0000 C CNN
+	1    9400 750
+	0    -1   -1   0
+$EndComp
+Wire Wire Line
+	9600 650  9400 650
+Wire Wire Line
+	9400 650  9400 700
+Connection ~ 9600 650
+$Comp
+L MLAB_MECHANICAL:HOLE M8
+U 1 1 5C71374D
+P 9200 750
+F 0 "M8" V 9100 750 60  0000 C CNN
+F 1 "BMI-S-204-F" H 9200 650 60  0001 C CNN
+F 2 "RF_Shielding:Laird_Technologies_BMI-S-204-F_32.00x32.00mm" H 9200 750 60  0001 C CNN
+F 3 "" H 9200 750 60  0000 C CNN
+	1    9200 750
+	0    -1   -1   0
+$EndComp
+Wire Wire Line
+	9400 650  9200 650
+Wire Wire Line
+	9200 650  9200 700
+Connection ~ 9400 650
 $EndSCHEMATC
