File: hw/sch_pcb/SPACEDOS01A_PCB01A/cpu.sch (KiCad schematic (older format))
At the start: 27 parts, among them J19 HEADER_2x01_PARALLEL, J22 HEADER_2x03, J4 HEADER_1x01, J5 HEADER_1x01, J6 HEADER_1x01, J7 HEADER_1x01, U10 ATMEGA1284P-AU, U11 PCF85263A, Y1 16MHz, Y2 ABS07-120-32.768KHZ-T

Commit message: Edit
Connections:
- net PB0: now reaches U10.40 ((PCINT8/T0/XCK)PB0)
- no-connect marks 24 -> 23
Changed lines of the file:
@@
 EESchema Schematic File Version 4
 LIBS:SPACEDOS01A_PCB01A-cache
-EELAYER 29 0
+EELAYER 26 0
 EELAYER END
 $Descr A4 11693 8268
@@
 NoConn ~ 6850 2600
 NoConn ~ 6850 2500
-NoConn ~ 6850 2400
 NoConn ~ 6850 2200
 NoConn ~ 6850 2100
@@
 NoConn ~ 6850 2800
 NoConn ~ 6850 3500
+Text GLabel 6950 2400 2    60   Input ~ 0
+PB0
+Wire Wire Line
+	6850 2400 6950 2400
 $EndSCHEMATC

Commit message: edit
Parts:
- Y1: footprint Mlab_XTAL:Crystal_HC49-U_Vertical -> Mlab_XTAL:Crystal_HC49-4H_Vertical
Changed lines of the file:
@@
 F 0 "Y1" H 2800 2568 50  0000 C CNN
 F 1 "16MHz" H 2800 2477 50  0000 C CNN
-F 2 "Mlab_XTAL:Crystal_HC49-U_Vertical" H 2800 2300 50  0001 C CNN
+F 2 "Mlab_XTAL:Crystal_HC49-4H_Vertical" H 2800 2300 50  0001 C CNN
 F 3 "~" H 2800 2300 50  0001 C CNN
 	1    2800 2300
