File: hw/sch_pcb/SPACEDOS01B_PCB01A/SPACEDOS01B_PCB01A.kicad_pcb (KiCad board)
At the start: 2 copper layers, 90.9 x 50.3 mm, 111 parts, among them J1 HEADER_2x01_PARALLEL, J19 HEADER_2x01_PARALLEL, J2 HEADER_2x01_PARALLEL, J22 HEADER_2x03, J3 HEADER_2x01_PARALLEL, J4 HEADER_1x01, J5 HEADER_1x01, J6 HEADER_1x01, J7 HEADER_1x01, M1 HOLE, M2 HOLE, M3 HOLE, M4 HOLE, M5 BMI-S-210-F, M6 BMI-S-210-F, M7 BMI-S-210-F, M8 BMI-S-204-F, U1 OPA2314, U10 ATMEGA1284P-AU, U11 PCF85263A, U2 OPA2314, U3 ISL21080DIH312Z-TK 1V25, U4 TS7211, U5 TS5A4594, U6 TPS613221ADBV, U8 TPS613222ADBV, Y1 16MHz, Y2 ABS07-120-32.768KHZ-T

Commit message: edit
Parts:
- moved C1 83.0 mm to (57.1, 61.2)
- moved C10 83.0 mm to (40.0, 53.6)
- moved C11 83.0 mm to (47.4, 53.7)
- moved C12 83.0 mm to (67.4, 52.6)
- moved C13 83.0 mm to (65.1, 44.5)
- moved C14 83.0 mm to (72.4, 60.6)
- moved C15 83.0 mm to (49.9, 50.1)
- moved C16 83.0 mm to (52.4, 50.0)
- moved C17 83.0 mm to (57.0, 49.2)
- moved C18 83.0 mm to (56.8, 53.7)
- moved C19 83.0 mm to (67.4, 48.8)
- moved C2 83.0 mm to (50.0, 42.9)
- moved C20 83.0 mm to (39.7, 57.9)
- moved C21 83.0 mm to (54.1, 42.9)
- moved C22 83.0 mm to (108.5, 64.4)
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
Commit message: edit
Parts:
- C1, C10, C11, C12, C13, C14, C15, C16, C17, C18, C19, C2, C20, C21, C22, C23, C24, C25, C26, C27, C28, C29, C3, C30, C31, C32, C33, C34, C35, C36, C38, C39, C4, C40, C42, C43, C44, C45, C47, C48, C49, C5, C50, C51, C52, C53, C54, C55, C6, C7, C8, C9, D1, D3, F1, F2, J22, L1, L2, L3, M6, M7, R1, R10, R11, R12, R13, R15, R19, R2, R20, R21, R22, R23, R24, R25, R27, R28, R3, R4, R5, R6, R7, R8, R9, U1, U10, U11, U2, U3, U4, U5, U6, U8, Y2: moved to F.Cu
- D2, J1, J19, J2, J3, J4, J5, J6, J7, M5, M8, Y1: moved to B.Cu
- moved M5 73.8 mm to (66.2, 110.2)
- moved C39 68.5 mm to (93.8, 107.5)
- moved R15 67.7 mm to (56.7, 107.1)
- moved R19 67.7 mm to (52.8, 107.1)
- moved R22 67.7 mm to (49.0, 107.1)
- moved C30 65.5 mm to (80.5, 106.0)
- moved C33 65.5 mm to (84.2, 106.0)
- moved J4 63.7 mm to (114.6, 105.1)
- moved J5 63.7 mm to (117.2, 105.1)
- moved C24 60.8 mm to (47.7, 103.6), turned to 90 degrees
- moved C2 60.6 mm to (50.0, 103.6), turned to 90 degrees
- moved C21 60.6 mm to (54.1, 103.6), turned to 90 degrees
- moved C23 60.6 mm to (52.0, 103.6), turned to 90 degrees
- moved Y1 60.6 mm to (80.0, 103.6)
- moved R1 60.6 mm to (72.0, 103.5), turned to 270 degrees
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Other:
- board size 90.9 x 50.3 mm -> 90.9 x 214.6 mm

Commit message: edit
Parts:
- removed C22, C38, C49: 10uF, Mlab_R:SMD-0805
- removed C25, C48, C53: 100nF, Mlab_R:SMD-0805
- removed C45, C51: NFM21PC105-1uF, Mlab_L:FIR1
- removed D1: BZV55C-5,6V, Diode_SMD:D_MiniMELF
- removed F1: SR010-15 100mA, Mlab_R:SMD-0805
- removed L2: DFE252012P-4R7M, Resistor_SMD:R_0805_2012Metric_Pad1.15x1.40mm_HandSolder
- removed R24, R25, R27: -, Mlab_R:SMD-0805
- removed R28: 0R, Mlab_R:SMD-0805
- removed U6: TPS613221ADBV, Package_TO_SOT_SMD:SOT-23-5
- added M10: BMI-S-204-F, RF_Shielding:Laird_Technologies_BMI-S-204-F_32.00x32.00mm, F.Cu at (221.0, -83.8)
- added M9: BMI-S-204-F, RF_Shielding:Laird_Technologies_BMI-S-204-F_32.00x32.00mm, F.Cu at (113.2, -72.5)
- moved J5 203.3 mm to (74.9, -93.8), turned to 90 degrees
- moved J7 201.3 mm to (72.4, -93.8), turned to 90 degrees
- moved J4 200.3 mm to (74.9, -91.2), turned to 90 degrees
- moved J6 198.3 mm to (72.4, -91.2), turned to 90 degrees
- moved J19 197.9 mm to (69.9, -92.5), turned to 90 degrees
- moved J2 196.1 mm to (67.3, -92.5), turned to 0 degrees
- moved J1 194.3 mm to (64.8, -92.5), turned to 0 degrees
- moved C43 192.6 mm to (70.9, -87.4), turned to 90 degrees
- moved J3 192.5 mm to (62.2, -92.5), turned to 0 degrees
- moved C28 191.0 mm to (68.7, -87.4), turned to 90 degrees
- moved C27 189.5 mm to (66.7, -87.4), turned to 90 degrees
- moved F2 189.0 mm to (58.8, -91.5), turned to 90 degrees
- moved C36 187.5 mm to (56.5, -91.5), turned to 90 degrees
- moved L1 187.3 mm to (71.8, -82.3), turned to 270 degrees
- moved C26 186.3 mm to (64.5, -86.1), turned to 90 degrees
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Connections:
- net /power/5 renamed Net-(J1-Pad1)
- C29 pad 3: Net-(C29-Pad3) -> +3V3
- C32 pad 1: VDD -> +3V3
- C55 pad 1: Net-(C29-Pad3) -> +3V3
- L3 pad 1: VDD -> +3V3
Routing:
- net +3V3: track 180.7 -> 199.5 mm
- net Net-(J1-Pad1): track 14.8 -> 2.54 mm
- net VDD: track 11.5 -> 0.00 mm
- net Net-(C45-Pad3): track 9.12 -> 0.00 mm
- net Net-(C38-Pad1): track 8.24 -> 0.00 mm
- net Net-(C29-Pad3): track 7.33 -> 0.00 mm
- net Net-(C22-Pad1): track 7.31 -> 0.00 mm
- net Net-(L2-Pad2): track 2.69 -> 0.00 mm
- net GND: track 133.6 -> 130.9 mm
- removed copper zone on B.Cu, net GND
- removed copper zone on F.Cu, net GND
Other:
- board size 90.9 x 214.6 mm -> 48.2 x 93.5 mm

Commit message: edit
Parts:
- removed C30, C33: 15pF, Mlab_R:SMD-0805
- removed M5, M7: BMI-S-210-F, Mlab_Mechanical:BMI-S-210-F
- removed Y1: 16MHz, Mlab_XTAL:Crystal_HC49-4H_Vertical
- M10: moved to B.Cu
- moved M10 165.1 mm to (58.2, -56.9), turned to 180 degrees
- moved M9 47.7 mm to (65.6, -68.9), turned to 90 degrees
- moved J5 35.1 mm to (79.5, -58.9)
- moved J7 33.1 mm to (79.5, -61.5)
- moved J4 32.4 mm to (77.0, -58.9)
- moved J6 30.1 mm to (77.0, -61.5)
- moved J19 29.7 mm to (78.2, -64.0), turned to 180 degrees
- moved J2 28.1 mm to (78.2, -66.5), turned to 270 degrees
- moved J1 27.0 mm to (78.2, -69.1), turned to 270 degrees
- moved F2 26.3 mm to (79.2, -75.0), turned to 270 degrees
- moved J3 26.3 mm to (78.2, -71.6), turned to 270 degrees
- moved C36 26.3 mm to (77.5, -75.7)
- moved D3 26.2 mm to (75.4, -76.2)
- moved C43 25.0 mm to (72.1, -62.5), turned to 0 degrees
- moved C29 23.1 mm to (78.2, -79.5), turned to 90 degrees
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Routing:
- net +3V3: track 199.5 -> 129.2 mm, vias 8 -> 6
- net /cpu/TX0: track 32.0 -> 0.00 mm, vias 2 -> 0
- net /cpu/RX0: track 29.1 -> 0.00 mm, vias 2 -> 0
- net GND: track 130.9 -> 106.2 mm, vias 193 -> 166
- net +5V: track 62.5 -> 38.4 mm, vias 2 -> 0
- net /cpu/PC3: track 21.4 -> 0.00 mm
- net /cpu/PC7: track 20.3 -> 0.00 mm
- net /cpu/RST#_P: track 34.6 -> 14.4 mm, vias 2 -> 1
- net Net-(C29-Pad1): track 12.5 -> 0.00 mm
- net Net-(C30-Pad1): track 11.1 -> 0.00 mm
- net /cpu/PC1: track 19.7 -> 10.4 mm, vias 2 -> 1
- net /cpu/PC0: track 21.7 -> 12.6 mm
- net /power/3: track 8.97 -> 0.00 mm
- net Net-(C33-Pad1): track 6.40 -> 0.00 mm
- net /cpu/RST#: track 5.82 -> 0.00 mm
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Other:
- outline, holes or cut-outs redrawn

Commit message: edit
Parts:
- moved C26 11.7 mm to (75.4, -81.8), turned to 270 degrees
- moved R21 9.39 mm to (54.0, -74.7), turned to 180 degrees
- moved C27 8.76 mm to (73.4, -81.8), turned to 270 degrees
- moved C28 6.12 mm to (71.1, -81.8), turned to 270 degrees
- moved C43 5.78 mm to (69.9, -57.1)
- moved C32 4.02 mm to (54.2, -67.1)
- moved L3 3.86 mm to (56.9, -64.8), turned to 180 degrees
- moved U8 3.51 mm to (53.1, -63.8)
- moved C50 3.45 mm to (55.6, -58.4)
- moved Y2 3.45 mm to (53.3, -78.2)
- moved C40 3.38 mm to (65.0, -80.3)
- moved C42 3.30 mm to (55.4, -60.7)
- moved L1 3.29 mm to (68.6, -81.5)
- moved C52 3.24 mm to (52.3, -56.6), turned to 270 degrees
- moved C31 2.95 mm to (68.8, -78.0), turned to 0 degrees
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Connections:
- J4 pad 1: /cpu/PC7 -> /cpu/PD3
- J5 pad 1: /cpu/PC3 -> /cpu/PD2
- U10 pad 11: (no net) -> /cpu/PD2
- U10 pad 12: (no net) -> /cpu/PD3
- U10 pad 22: /cpu/PC3 -> (no net)
- U10 pad 26: /cpu/PC7 -> (no net)
- U10 pad 7: Net-(C30-Pad1) -> (no net)
- U10 pad 8: Net-(C33-Pad1) -> (no net)
Routing:
- net +3V3: track 129.2 -> 200.7 mm
- net /cpu/PD2: track 0.00 -> 16.0 mm, vias 0 -> 2
- net /cpu/PC1: track 10.4 -> 23.7 mm, vias 1 -> 2
- net /cpu/PC0: track 12.6 -> 25.8 mm
- net /cpu/TX0: track 0.00 -> 12.3 mm
- net /cpu/RST#: track 0.00 -> 11.5 mm, vias 0 -> 2
- net /cpu/PD3: track 0.00 -> 11.1 mm, vias 0 -> 2
- net GND: track 106.2 -> 95.5 mm, vias 166 -> 158
- net /cpu/RX0: track 0.00 -> 9.89 mm
- net Net-(C29-Pad1): track 0.00 -> 8.04 mm
- net +5V: track 38.4 -> 46.1 mm
- net /power/3: track 0.00 -> 5.06 mm
- net Net-(U11-Pad2): track 0.00 -> 2.59 mm
- net Net-(U11-Pad1): track 0.00 -> 2.58 mm
- net Net-(J1-Pad1): track 0.00 -> 2.54 mm
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- added copper zone on B.Cu, net GND
- added copper zone on F.Cu, net GND

Commit message: edit PCB
Parts:
- removed D2: S2744-09, Mlab_D:HAMAMATSU_S2744-09
- added D1: S11773-02, Mlab_D:HAMAMATSU_S11773-02, F.Cu at (74.2, -17.6)
- moved C4 7.01 mm to (58.7, -37.1), turned to 0 degrees
- moved R7 1.12 mm to (68.8, -22.2), turned to 270 degrees
- moved C3 0.82 mm to (68.0, -11.5)
- moved R8 0.80 mm to (69.8, -25.0)
- moved R9 0.29 mm to (66.0, -24.2)
- moved C11 0.23 mm to (62.5, -24.0)
- moved C6 0.23 mm to (62.5, -26.0)
Routing:
- net GND: track 95.5 -> 105.5 mm, vias 158 -> 162
- net /cpu/RST#: track 11.5 -> 14.1 mm
- net +3V3: track 200.7 -> 199.5 mm
- net /A: track 16.1 -> 17.2 mm
- net PA1: track 104.1 -> 105.2 mm
- net /K: track 5.94 -> 6.78 mm
- net Net-(C15-Pad2): track 8.86 -> 9.45 mm
Other:
- board text added: "PD2"
- board text added: "PD3"
- board text added: "SPACEDOS01B_PCB01A"
- board text removed: "5V"
- board text removed: "PC3"
- board text removed: "PC7"
- board text removed: "SPACEDOS01A_PCB01A"

Commit message: edit
Parts:
- C1: value 47uF -> 22uF
- C29, C52: footprint Mlab_L:FIR1 -> Mlab_L:FIR_0805
- F2: value SR010-15 100mA -> 2R2
- J1: value HEADER_2x01_PARALLEL -> HEADER_2x01
- turned J1 to 90 degrees
Connections:
- J1 pad 1: Net-(J1-Pad1) -> (no net)
- J1 pad 2: Net-(J1-Pad1) -> (no net)
Routing:
- net Net-(J1-Pad1): track 2.54 -> 0.00 mm
- net GND: track 105.5 -> 106.2 mm
Other:
- board text added: "PB6"
- board text added: "RX"
- board text added: "TX"
