File: hw/sch_pcb/SPACEDOS01B_PCB01A/SPACEDOS01B_PCB01A.kicad_pcb (KiCad board)
At the start: 2 copper layers, 48.2 x 93.5 mm, 92 parts, among them J1 HEADER_2x01, J19 HEADER_2x01_PARALLEL, J2 HEADER_2x01_PARALLEL, J22 HEADER_2x03, J3 HEADER_2x01_PARALLEL, J4 HEADER_1x01, J5 HEADER_1x01, J6 HEADER_1x01, J7 HEADER_1x01, M1 HOLE, M10 BMI-S-204-F, M2 HOLE, M3 HOLE, M4 HOLE, M6 BMI-S-210-F, M8 BMI-S-204-F, M9 BMI-S-204-F, U1 OPA2314, U10 ATMEGA1284P-AU, U11 PCF85263A, U2 OPA2314, U3 ISL21080DIH312Z-TK 1V25, U4 TS7211, U5 TS5A4594, U8 TPS613222ADBV, Y2 ABS07-120-32.768KHZ-T

Commit message: Center PCB in page. Improve dimensions.
Parts:
- moved M1 235.3 mm to (181.7, 122.5), turned to -90 degrees
- moved C55 222.8 mm to (173.7, 118.7), turned to -90 degrees
- moved C26 219.9 mm to (172.7, 115.4), turned to 180 degrees
- moved C27 219.0 mm to (172.7, 113.4), turned to 180 degrees
- moved C29 218.1 mm to (170.4, 118.2), turned to 0 degrees
- moved C28 218.0 mm to (172.7, 111.1), turned to 180 degrees
- moved L1 216.6 mm to (172.5, 108.6), turned to 180 degrees
- moved D3 214.2 mm to (169.2, 113.4), turned to 90 degrees
- moved C40 213.5 mm to (171.2, 104.9), turned to -90 degrees
- moved F2 212.7 mm to (165.9, 119.2), turned to 180 degrees
- moved C31 211.9 mm to (168.9, 108.8), turned to -90 degrees
- moved C47 211.5 mm to (171.7, 96.9), turned to 90 degrees
- moved C36 211.5 mm to (165.9, 116.9), turned to 180 degrees
- moved R20 210.9 mm to (170.1, 101.7), turned to 0 degrees
- moved C44 210.6 mm to (168.9, 105.4), turned to -90 degrees
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Other:
- board size 48.2 x 93.5 mm -> 93.5 x 48.2 mm
