File: hw/sch_pcb/SPACEDOS01B_PCB01A/SPACEDOS01B_PCB01A.sch (KiCad schematic (older format))
At the start: 53 parts, among them M1 HOLE, M2 HOLE, M3 HOLE, M4 HOLE, M5 BMI-S-210-F, M6 BMI-S-210-F, M7 BMI-S-210-F, M8 BMI-S-204-F, U1 OPA2314, U2 OPA2314, U3 ISL21080DIH312Z-TK 1V25, U4 TS7211, U5 TS5A4594

Commit message: edit
Parts:
- added M10, M9: BMI-S-204-F, RF_Shielding:Laird_Technologies_BMI-S-204-F_32.00x32.00mm, symbol MLAB_MECHANICAL:HOLE
Connections:
- net GND: now also M10.1, M9.1
Changed lines of the file:
@@
 	9200 650  9200 700
 Connection ~ 9400 650
+$Comp
+L MLAB_MECHANICAL:HOLE M9
+U 1 1 5C81F263
+P 8800 750
+F 0 "M9" V 8700 750 60  0000 C CNN
+F 1 "BMI-S-204-F" H 8800 650 60  0001 C CNN
+F 2 "RF_Shielding:Laird_Technologies_BMI-S-204-F_32.00x32.00mm" H 8800 750 60  0001 C CNN
+F 3 "" H 8800 750 60  0000 C CNN
+	1    8800 750
+	0    -1   -1   0
+$EndComp
+$Comp
+L MLAB_MECHANICAL:HOLE M10
+U 1 1 5C81F2E9
+P 9000 750
+F 0 "M10" V 8900 750 60  0000 C CNN
+F 1 "BMI-S-204-F" H 9000 650 60  0001 C CNN
+F 2 "RF_Shielding:Laird_Technologies_BMI-S-204-F_32.00x32.00mm" H 9000 750 60  0001 C CNN
+F 3 "" H 9000 750 60  0000 C CNN
+	1    9000 750
+	0    -1   -1   0
+$EndComp
+Wire Wire Line
+	9200 650  9000 650
+Wire Wire Line
+	8800 650  8800 700
+Connection ~ 9200 650
+Wire Wire Line
+	9000 700  9000 650
+Connection ~ 9000 650
+Wire Wire Line
+	9000 650  8800 650
 $EndSCHEMATC

Commit message: edit
Parts:
- removed M7: BMI-S-210-F, Mlab_Mechanical:BMI-S-210-F, symbol MLAB_MECHANICAL:HOLE
Changed lines of the file:
@@
 EESchema Schematic File Version 4
 LIBS:SPACEDOS01B_PCB01A-cache
-EELAYER 26 0
+EELAYER 29 0
 EELAYER END
 $Descr A4 11693 8268
@@
 Wire Wire Line
 	2200 7200 2200 7150
-$Comp
-L MLAB_MECHANICAL:HOLE M7
-U 1 1 5C564E7A
-P 9600 750
-F 0 "M7" V 9500 750 60  0000 C CNN
-F 1 "BMI-S-210-F" H 9600 650 60  0001 C CNN
-F 2 "Mlab_Mechanical:BMI-S-210-F" H 9600 750 60  0001 C CNN
-F 3 "" H 9600 750 60  0000 C CNN
-	1    9600 750
-	0    -1   -1   0
-$EndComp
-Wire Wire Line
-	9600 650  9600 700
-Wire Wire Line
-	9600 650  10000 650
 Wire Wire Line
 	8350 5150 10550 5150
@@
 $EndComp
 Wire Wire Line
-	9600 650  9400 650
-Wire Wire Line
 	9400 650  9400 700
-Connection ~ 9600 650
 $Comp
 L MLAB_MECHANICAL:HOLE M8
@@
 Wire Wire Line
 	9000 650  8800 650
+Wire Wire Line
+	9400 650  10000 650
 $EndSCHEMATC

Commit message: edit
Parts:
- removed M5: BMI-S-210-F, Mlab_Mechanical:BMI-S-210-F, symbol MLAB_MECHANICAL:HOLE
Changed lines of the file:
@@
 Text GLabel 10550 5150 2    60   Input ~ 0
 PB0
-$Comp
-L MLAB_MECHANICAL:HOLE M5
-U 1 1 5C7015D6
-P 9400 750
-F 0 "M5" V 9300 750 60  0000 C CNN
-F 1 "BMI-S-210-F" H 9400 650 60  0001 C CNN
-F 2 "Mlab_Mechanical:BMI-S-210-F" H 9400 750 60  0001 C CNN
-F 3 "" H 9400 750 60  0000 C CNN
-	1    9400 750
-	0    -1   -1   0
-$EndComp
 Wire Wire Line
 	9400 650  9400 700

Commit message: edit PCB
Parts:
- removed D2: S2744-09, Mlab_D:HAMAMATSU_S2744-09, symbol Device:D_Photo
- added D1: S11773-02, Mlab_D:HAMAMATSU_S11773-02, symbol Device:D_Photo
Connections:
- net A: now also D1.2 (A)
- net K: now also D1.1 (K)
Changed lines of the file:
@@
 Wire Wire Line
 	1750 4950 1900 4950
-$Comp
-L Device:D_Photo D2
-U 1 1 5B3A05A5
-P 1700 4350
-F 0 "D2" H 1650 4645 50  0000 C CNN
-F 1 "S2744-09" H 1650 4554 50  0000 C CNN
-F 2 "Mlab_D:HAMAMATSU_S2744-09" H 1650 4350 50  0001 C CNN
-F 3 "~" H 1650 4350 50  0001 C CNN
-	1    1700 4350
-	1    0    0    -1
-$EndComp
 Text Label 1500 4950 0    60   ~ 0
 REF
@@
 	1800 4350 1900 4350
 Connection ~ 1900 4350
-Wire Wire Line
-	1900 4350 1900 4750
 $Sheet
 S 6750 800  850  350
@@
 Text Label 1000 4350 0    60   ~ 0
 Ubiasout
-Wire Wire Line
-	1000 4350 1500 4350
 $Comp
 L power:+3.3V #PWR0106
@@
 Wire Wire Line
 	9400 650  10000 650
+$Comp
+L Device:D_Photo D1
+U 1 1 5C80A3E9
+P 1700 4350
+F 0 "D1" H 1350 4450 50  0000 C CNN
+F 1 "S11773-02" H 1650 4550 50  0000 C CNN
+F 2 "Mlab_D:HAMAMATSU_S11773-02" H 1650 4350 50  0001 C CNN
+F 3 "~" H 1650 4350 50  0001 C CNN
+	1    1700 4350
+	1    0    0    -1
+$EndComp
+Wire Wire Line
+	1900 4350 1900 4750
+Wire Wire Line
+	1000 4350 1500 4350
 $EndSCHEMATC

Commit message: edit
Parts:
- C1: value 47uF -> 22uF
Changed lines of the file:
@@
 EESchema Schematic File Version 4
 LIBS:SPACEDOS01B_PCB01A-cache
-EELAYER 29 0
+EELAYER 26 0
 EELAYER END
 $Descr A4 11693 8268
@@
 P 1400 1150
 F 0 "C1" H 1518 1196 50  0000 L CNN
-F 1 "47uF" H 1518 1105 50  0000 L CNN
+F 1 "22uF" H 1518 1105 50  0000 L CNN
 F 2 "Mlab_C:TantalC_SizeC_Reflow" H 1438 1000 50  0001 C CNN
 F 3 "~" H 1400 1150 50  0001 C CNN
@@
 Text GLabel 10550 5150 2    60   Input ~ 0
 PB0
-Wire Wire Line
-	9400 650  9400 700
 $Comp
 L MLAB_MECHANICAL:HOLE M8
@@
 $EndComp
 Wire Wire Line
-	9400 650  9200 650
-Wire Wire Line
 	9200 650  9200 700
-Connection ~ 9400 650
 $Comp
 L MLAB_MECHANICAL:HOLE M9
@@
 Wire Wire Line
 	9000 650  8800 650
-Wire Wire Line
-	9400 650  10000 650
 $Comp
 L Device:D_Photo D1
@@
 Wire Wire Line
 	1000 4350 1500 4350
+Wire Wire Line
+	9200 650  10000 650
 $EndSCHEMATC
